File: devboard/cisco_hwic_dev_board/cisco_hwic_dev_board.kicad_pcb (KiCad board)
At the start: 2 copper layers, 3 parts, among them J1 Cisco_HWIC, J2 Conn_02x17_Odd_Even, J3 Conn_02x17_Odd_Even

Commit message: Rename.
Parts:
- J1: footprint cisc_hwic_dev_board:PinHeader_2x34_P1.27mm_Vertical_SMD_Top_Bottom -> cisco_hwic_dev_board:PinHeader_2x34_P1.27mm_Vertical_SMD_Top_Bottom
Changed lines of the file:
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@@
     (0 F.Cu signal)
     (31 B.Cu signal)
-    (32 B.Adhes user hide)
-    (33 F.Adhes user hide)
-    (34 B.Paste user hide)
-    (35 F.Paste user hide)
-    (36 B.SilkS user hide)
-    (37 F.SilkS user hide)
-    (38 B.Mask user hide)
-    (39 F.Mask user hide)
-    (40 Dwgs.User user hide)
-    (41 Cmts.User user hide)
-    (42 Eco1.User user hide)
-    (43 Eco2.User user hide)
-    (44 Edge.Cuts user hide)
-    (45 Margin user hide)
-    (46 B.CrtYd user hide)
-    (47 F.CrtYd user hide)
-    (48 B.Fab user hide)
-    (49 F.Fab user hide)
+    (32 B.Adhes user)
+    (33 F.Adhes user)
+    (34 B.Paste user)
+    (35 F.Paste user)
+    (36 B.SilkS user)
+    (37 F.SilkS user)
+    (38 B.Mask user)
+    (39 F.Mask user)
+    (40 Dwgs.User user)
+    (41 Cmts.User user)
+    (42 Eco1.User user)
+    (43 Eco2.User user)
+    (44 Edge.Cuts user)
+    (45 Margin user)
+    (46 B.CrtYd user)
+    (47 F.CrtYd user)
+    (48 B.Fab user)
+    (49 F.Fab user)
   )
   (setup
@@
     (add_net "Net-(J2-Pad7)")
   )
-  (module cisc_hwic_dev_board:PinHeader_2x34_P1.27mm_Vertical_SMD_Top_Bottom (layer F.Cu)
+  (module cisco_hwic_dev_board:PinHeader_2x34_P1.27mm_Vertical_SMD_Top_Bottom (layer F.Cu)
     (at -541.02 -538.48)
     (descr "surface-mounted straight pin header, 2x34, 1.27mm pitch, double rows")
@@
       (effects (font (size 1 1) (thickness 0.15)))
     )
+    (fp_text user 12V (at -5.715 -3.81) (layer B.SilkS)
+      (effects (font (size 1 1) (thickness 0.15)) (justify mirror))
+    )
+    (fp_text user GND (at -5.485 -6.35) (layer F.SilkS)
+      (effects (font (size 1 1) (thickness 0.15)))
+    )
+    (fp_text user 5V (at -4.826 -13.97) (layer F.SilkS)
+      (effects (font (size 1 1) (thickness 0.15)))
+    )
+    (fp_text user 3.3V (at -5.485 -8.89) (layer F.SilkS)
+      (effects (font (size 1 1) (thickness 0.15)))
+    )
     (fp_text user 12V (at -5.485 -3.81) (layer F.SilkS)
-      (effects (font (size 1 1) (thickness 0.15)))
-    )
-    (fp_text user GND (at -5.485 -6.35) (layer F.SilkS)
-      (effects (font (size 1 1) (thickness 0.15)))
-    )
-    (fp_text user 5V (at -5.715 -13.97) (layer B.SilkS)
-      (effects (font (size 1 1) (thickness 0.15)) (justify mirror))
-    )
-    (fp_text user 3.3V (at -5.715 -8.89) (layer B.SilkS)
-      (effects (font (size 1 1) (thickness 0.15)) (justify mirror))
-    )
-    (fp_text user 12V (at -5.485 -3.81) (layer F.SilkS)
