File: devboard/cisco_hwic_dev_board/cisco_hwic_dev_board.sch (KiCad schematic (older format))
At the start: 3 parts, among them J1 Cisco_HWIC, J2 Conn_02x17_Odd_Even, J3 Conn_02x17_Odd_Even

Commit message: Rename.
Parts:
- J1: footprint cisc_hwic_dev_board:PinHeader_2x34_P1.27mm_Vertical_SMD_Top_Bottom -> cisco_hwic_dev_board:PinHeader_2x34_P1.27mm_Vertical_SMD_Top_Bottom
Changed lines of the file:
@@
 F 0 "J1" H 4600 5067 50  0000 C CNN
 F 1 "Cisco_HWIC" H 4600 4976 50  0000 C CNN
-F 2 "cisc_hwic_dev_board:PinHeader_2x34_P1.27mm_Vertical_SMD_Top_Bottom" H 4550 3250 50  0001 C CNN
+F 2 "cisco_hwic_dev_board:PinHeader_2x34_P1.27mm_Vertical_SMD_Top_Bottom" H 4550 3250 50  0001 C CNN
 F 3 "~" H 4550 3250 50  0001 C CNN
 	1    4550 3250
